Commit message: 重大修改

File: models/05_urdf/urdf/05_urdf_temp.urdf (robot description, URDF)
Before this commit: robot 05_urdf, 9 links, 8 joints
Joints:
- joint end_joint: origin xyz=0.076 0 0 rpy=0 0 0 -> xyz=0.08181 0 0 rpy=0 0 0
- joint joint1: origin xyz=0 0 0.2015 rpy=0 0 0 -> xyz=0 0 0.217 rpy=0 0 0
- joint joint2: axis 0 0 -1 -> 0 0 1
- joint joint3: origin xyz=0 -0.268 0 rpy=1.5708 0 0 -> xyz=0 -0.28493 0 rpy=1.5708 0 0
- joint joint5: origin xyz=0 0.204 0 rpy=-1.5708 0 0 -> xyz=0 0.221 0 rpy=-1.5708 0 0
- joint joint6: origin xyz=0 0 0 rpy=-1.5708 0 0 -> xyz=0 0 0 rpy=-1.5708 -1.5708 0
- joint joint7: origin xyz=-0.001 -0.088 0 rpy=-1.5708 0 -1.5708 -> xyz=0.08365 0 0 rpy=-1.5708 0 0
